File: HOMADOS.sch (EAGLE design)
At the start: 72 parts, among them P1 39-30-02, P10 39-30-02, P11 39-30-02, P12 39-30-02, P13 39-30-02, P14 39-30-02, P15 39-30-02, P16 39-30-02, P17 39-30-02, P2 39-30-02, P3 39-30-02, P4 39-30-02, P5 39-30-02, P6 39-30-02, P7 39-30-02, P8 39-30-02, P9 39-30-02, Q1 T460, Q10 T460, Q11 T460, Q12 T460, Q13 T460, Q14 T460, Q15 T460, Q16 T460, Q2 T460, Q3 T460, Q4 T460, Q5 T460, Q6 T460, Q7 T460, Q8 T460, Q9 T460, U1 ARDUINO-MEGA-SOLINOID

Commit message: created v2 of Homados board
Parts:
- removed LED1, LED2: (no value), adafruit:LED5MM
- removed U1: ARDUINO-MEGA-SOLINOID, Nathans-Arduinos2:ARDUINO-MEGA-SOLINOID
- added I2C-1, I2C-2, I2C-3: JST-PH_4-PIN_HEADER, JST_connectors:JST-PH_4-PIN_HEADER
- added P18: 39-30-02, con-molex-mini-fit:39-30-02
- added R19: 1k, SparkFun-Passives:RESISTORKIT
- added R20, R21: 100, SparkFun-Passives:RESISTORKIT
- added U$2: RGBLED_CA, adafruit:RGBLED_CA
- added U2: ARDUINO-MEGAPRO-5V, SparkFun-Minimal-Shields:ARDUINO-MEGAPRO-5V
- R1, R2: value 1k -> 4.7k
- R3: value 1k -> 180
Connections:
- removed net D10: R17.1, U1.32(PC5)
- removed net D12: R18.1, U1.34
- removed net D2: R13.1, U1.24(PA2)
- removed net D4: R14.1, U1.26(PA4)
- removed net D6: R15.1, U1.28(PA6)
- removed net D8: R16.1, U1.30(PC7)
- removed net N$5: U1.13(PB7)
- new net 5V: I2C-1.4, I2C-2.4, I2C-3.4, R1.2, R2.1, U2.5V@1, U2.5V@2
- new net A0: R3.1, U$2.BLUE
- new net A2: R20.1, U$2.RED
- new net ARDUINO_GND: U$2.VCC, U2.GND@2
- new net BLUE: R3.2, U2.42
- new net GREEN: R21.2, U2.40
- new net N$12: U2.18(TX1)
- new net N$13: U2.19(RX1)
- new net N$17: U2.43
- new net N$28: U2.48
- new net N$29: U2.49
- new net N$32: U2.50
- new net N$6: Q1.B, R19.2
- new net N$8: U2.16(TX2)
- new net N$9: U2.17(RX2)
- new net N23: U2.51
- new net N24: U2.52
- new net N25: U2.53
- new net PW11: R9.1, U2.13
- new net PW12: R18.1, U2.44
- new net PW13: R17.1, U2.45
- new net PW14: R16.1, U2.46
- new net RED: R20.2, U2.41
- new net SCL: I2C-1.2, I2C-2.2, I2C-3.2, R2.2, U2.21(SCL)
- new net SDA: I2C-1.3, I2C-2.3, I2C-3.3, R1.1, U2.20(SDA)
- net D0: now also R15.1, U2.47; no longer R12.1, U1.22(PA0)
- net GND: now also I2C-1.1, I2C-2.1, I2C-3.1, P18.2, Q1.C, Q10.C, Q11.C, Q12.C, Q13.C, Q14.C, Q15.C, Q16.C, Q2.C, Q3.C, Q4.C, Q5.C, Q6.C, Q7.C, Q8.C, Q9.C, U2.GND@3, U2.GND@4; no longer Q1.E, Q10.E, Q11.E, Q12.E, Q13.E, Q14.E, Q15.E, Q16.E, Q2.E, Q3.E, Q4.E, Q5.E, Q6.E, Q7.E, Q8.E, Q9.E, R1.2, R3.2, U1.GND@0, U1.GND@1, U1.GND@2, U1.GND@3, U1.GND@4
- net N$1: now also R21.1, U$2.GREEN; no longer LED1.C, R1.1
- net N$11: now also Q3.E; no longer Q3.C
- net N$15: now also Q4.E; no longer Q4.C
- net N$19: now also Q8.E; no longer Q5.C
- net N$2: now also Q1.E; no longer Q1.C
- net N$22: now also Q8.B; no longer Q5.B
- net N$23: now also Q7.E; no longer Q6.C
- net N$26: now also Q7.B; no longer Q6.B
- net N$27: now also Q6.E; no longer Q7.C
- net N$3: now also U2.14(TX3); no longer LED2.C, R3.1
- net N$30: now also Q6.B; no longer Q7.B
- net N$31: now also Q5.E; no longer Q8.C
- net N$34: now also Q5.B; no longer Q8.B
- net N$35: now also Q12.E; no longer Q9.C
- net N$38: now also Q12.B; no longer Q9.B
- net N$39: now also Q11.E; no longer Q10.C
- net N$4: now also Q2.E; no longer Q2.C
- net N$42: now also Q11.B; no longer Q10.B
- net N$43: now also Q10.E; no longer Q11.C
- net N$46: now also Q10.B; no longer Q11.B
- net N$47: now also Q9.E; no longer Q12.C
- net N$50: now also Q9.B; no longer Q12.B
- net N$51: now also Q16.E; no longer Q13.C
- net N$54: now also Q16.B; no longer Q13.B
- net N$55: now also Q15.E; no longer Q14.C
- net N$58: now also Q15.B; no longer Q14.B
- net N$59: now also Q14.E; no longer Q15.C
- net N$62: now also Q14.B; no longer Q15.B
- net N$63: now also Q13.E; no longer Q16.C
- net N$66: now also Q13.B; no longer Q16.B
- net N$7: now also U2.15(RX3); no longer Q1.B, R2.2
- net PW0: now also R14.1, U2.2; no longer R2.1, U1.2(PE4)
- net PW1: now also R13.1, U2.3; no longer R4.1, U1.3(PE5)
- net PW10: now also R10.1, U2.12; no longer LED2.A, U1.12(PB6)
- net PW2: now also R12.1, U2.4; no longer R5.1, U1.4(PG5)
- net PW3: now also R19.1, U2.5; no longer R6.1, U1.5(PE3)
- net PW4: now also R4.1, U2.6; no longer R7.1, U1.6(PH3)
- net PW5: now also R5.1, U2.7; no longer R8.1, U1.7(PH4)
- net PW6: now also R6.1, U2.8; no longer R9.1, U1.8(PH5)
- net PW7: now also R7.1, U2.9; no longer R10.1, U1.9(PH6)
- net PW8: now also R8.1, U2.10; no longer R11.1, U1.10(PB4)
- net PW9: now also R11.1, U2.11; no longer LED1.A, U1.11(PB5)
- net PWR: now also P18.1
Other:
- note added: "2x I2C busses"
- note added: "I2C"
- note added: "Power Rail on Single Side"
- note added: "connectors need to all be in row"
- note added: "find better package for mosfets,"
- note added: "mosfets are far too close to each other"
- note added: "new shield that keeps pins 44-gnd,"
- note added: "use all PWM pins instead of random digital pins"
- moved on the sheet: Q1, Q10, Q11, Q12, Q13, Q14, Q15, Q16, Q2, Q3, Q4, Q5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
