File: pcb/EAGLE/HOMADOS.sch (EAGLE design)
At the start: 78 parts, among them P1 39-30-02, P10 39-30-02, P11 39-30-02, P12 39-30-02, P13 39-30-02, P14 39-30-02, P15 39-30-02, P16 39-30-02, P17 39-30-02, P18 39-30-02, P2 39-30-02, P3 39-30-02, P4 39-30-02, P5 39-30-02, P6 39-30-02, P7 39-30-02, P8 39-30-02, P9 39-30-02, Q1 T460, Q10 T460, Q11 T460, Q12 T460, Q13 T460, Q14 T460, Q15 T460, Q16 T460, Q2 T460, Q3 T460, Q4 T460, Q5 T460, Q6 T460, Q7 T460, Q8 T460, Q9 T460, U2 ARDUINO-MEGAPRO-5V

Commit message: finished revision of homados
Parts:
- removed Q16: T460, transistor-npn:MJE800
- added Q17: (no value), transistor-power:PMOSFET_NTO220BV
- Q1, Q10, Q11, Q12, Q13, Q14, Q15, Q2, Q3, Q4, Q5, Q6, Q7, Q8, Q9: value T460 -> (none); device transistor-npn:MJE800 -> transistor-power:PMOSFET_NTO220BV
- renumbered P2 to P19
Connections:
- removed net N$39: D10.A, P11.2, Q11.E
- removed net N$43: D11.A, P12.2, Q10.E
- removed net N$47: D12.A, P13.2, Q9.E
- removed net N$51: D13.A, P14.2, Q16.E
- removed net N$55: D14.A, P15.2, Q15.E
- removed net N$59: D15.A, P16.2, Q14.E
- removed net N$63: D16.A, P17.2, Q13.E
- new net N$16: D3.A, P4.2, Q2.D
- new net N$20: D6.A, P7.2, Q6.D
- new net N$21: D7.A, P8.2, Q5.D
- new net N$24: D14.A, P15.2, Q14.D
- new net N$25: D15.A, P16.2, Q13.D
- new net N$33: D10.A, P11.2, Q9.D
- new net N$5: D12.A, P13.2, Q11.D
- net GND: now also Q1.S, Q10.S, Q11.S, Q12.S, Q13.S, Q14.S, Q15.S, Q17.S, Q2.S, Q3.S, Q4.S, Q5.S, Q6.S, Q7.S, Q8.S, Q9.S; no longer Q1.C, Q10.C, Q11.C, Q12.C, Q13.C, Q14.C, Q15.C, Q16.C, Q2.C, Q3.C, Q4.C, Q5.C, Q6.C, Q7.C, Q8.C, Q9.C
- net N$10: now also Q1.G; no longer Q2.B
- net N$11: now also D13.A, P14.2, Q15.D; no longer D3.A, P4.2, Q3.E
- net N$14: now also Q2.G; no longer Q3.B
- net N$15: now also D1.A, P1.2, Q1.D; no longer D4.A, P5.2, Q4.E
- net N$18: now also Q3.G; no longer Q4.B
- net N$19: now also D4.A, P5.2, Q3.D; no longer D5.A, P6.2, Q8.E
- net N$2: now also Q17.D; no longer Q1.E
- net N$22: now also Q7.G; no longer Q8.B
- net N$23: now also D11.A, P12.2, Q10.D; no longer D6.A, P7.2, Q7.E
- net N$26: now also Q6.G; no longer Q7.B
- net N$27: now also D8.A, P9.2, Q4.D; no longer D7.A, P8.2, Q6.E
- net N$30: now also Q5.G; no longer Q6.B
- net N$31: now also D16.A, P17.2, Q12.D; no longer D8.A, P9.2, Q5.E
- net N$34: now also Q4.G; no longer Q5.B
- net N$35: now also Q8.D; no longer Q12.E
- net N$38: now also Q8.G; no longer Q12.B
- net N$4: now also D5.A, P6.2, Q7.D; no longer D1.A, P1.2, Q2.E
- net N$42: now also Q9.G; no longer Q11.B
- net N$46: now also Q10.G; no longer Q10.B
- net N$50: now also Q11.G; no longer Q9.B
- net N$54: now also Q15.G; no longer Q16.B
- net N$58: now also Q14.G; no longer Q15.B
- net N$6: now also Q17.G; no longer Q1.B
- net N$62: now also Q13.G; no longer Q14.B
- net N$66: now also Q12.G; no longer Q13.B
Other:
- note added: "Power Connectors"
- note removed: "2x I2C busses"
- note removed: "Power Connector"
- note removed: "Power Rail on Single Side"
- note removed: "connectors need to all be in row"
- note removed: "find better package for mosfets,"
- note removed: "mosfets are far too close to each other"
- note removed: "new shield that keeps pins 44-gnd,"
- note removed: "use all PWM pins instead of random digital pins"
- moved on the sheet: D1, D10, D11, D12, D13, D14, D15, D16, D2, D3, D4, D5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

Commit message: added some specialized firmware
Connections:
- removed net N$17: U2.43
- removed net N$28: U2.48
- removed net N$29: U2.49
- removed net N$32: U2.50
- removed net N23: U2.51
- removed net N24: U2.52
- removed net N25: U2.53
Changed lines of the file:
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@@
-</segment>
-</net>
-<net name="N$17" class="0">
-<segment>
-<pinref part="U2" gate="G$1" pin="43"/>
-<wire x1="27.94" y1="60.96" x2="30.48" y2="60.96" width="0.1524" layer="91"/>
-<label x="30.48" y="60.96" size="1.27" layer="95" xref="yes"/>
-</segment>
-</net>
-<net name="N$28" class="0">
-<segment>
-<pinref part="U2" gate="G$1" pin="48"/>
-<wire x1="27.94" y1="48.26" x2="30.48" y2="48.26" width="0.1524" layer="91"/>
-<label x="30.48" y="48.26" size="1.27" layer="95" xref="yes"/>
-</segment>
-</net>
-<net name="N$29" class="0">
-<segment>
-<pinref part="U2" gate="G$1" pin="49"/>
-<wire x1="27.94" y1="45.72" x2="30.48" y2="45.72" width="0.1524" layer="91"/>
-<label x="30.48" y="45.72" size="1.27" layer="95" xref="yes"/>
-</segment>
-</net>
-<net name="N$32" class="0">
-<segment>
-<pinref part="U2" gate="G$1" pin="50"/>
-<wire x1="27.94" y1="43.18" x2="30.48" y2="43.18" width="0.1524" layer="91"/>
-<label x="30.48" y="43.18" size="1.27" layer="95" xref="yes"/>
 </segment>
 </net>
@@
 </segment>
 </net>
-<net name="N23" class="0">
-<segment>
-<pinref part="U2" gate="G$1" pin="51"/>
-<wire x1="27.94" y1="40.64" x2="30.48" y2="40.64" width="0.1524" layer="91"/>
-<label x="30.48" y="40.64" size="1.27" layer="95" xref="yes"/>
-</segment>
-</net>
-<net name="N24" class="0">
-<segment>
-<pinref part="U2" gate="G$1" pin="52"/>
-<wire x1="27.94" y1="38.1" x2="30.48" y2="38.1" width="0.1524" layer="91"/>
-<label x="30.48" y="38.1" size="1.27" layer="95" xref="yes"/>
-</segment>
-</net>
-<net name="N25" class="0">
-<segment>
-<pinref part="U2" gate="G$1" pin="53"/>
-<wire x1="27.94" y1="35.56" x2="30.48" y2="35.56" width="0.1524" layer="91"/>
-<label x="30.48" y="35.56" size="1.27" layer="95" xref="yes"/>
-</segment>
-</net>
